File: canda.kicad_sch (KiCad schematic)
At the start: 47 parts, among them J1 2s_cortex-m-10-pin, J3 2x4 male header 2.54 mm, J4 Conn_header_01x04_THT_2.54mm, J5 Screw_Terminal_01x02, J6 Screw_Terminal_01x02, M1 Motor_Servo, Q1 BSS138, Q2 DMG2305UX-13, U1 TPS613222ADBZ, U2 TLV75533PDBVR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

Commit message: updates
Parts:
- removed Q2: DMG2305UX-13, Package_TO_SOT_SMD:SOT-23-3, symbol 2s_transistors:DMG2305UX-13
- added Q3: DMG2305UX-13, Package_TO_SOT_SMD:SOT-23-3, symbol 2s_transistors:DMG2305UX-13
Connections:
- net +BATT: now also Q3.2 (S)
- net at Q1.3 (D), R6.2: now also Q3.1 (G)
- net at C7.1, L2.1: now also Q3.3 (D)

Commit message: ?
Parts:
- removed R11: 47k_0805, Resistor_SMD:R_0805_2012Metric, symbol 2s_Resistor_0805:47k_0805
- added R13: 47k_0805, Resistor_SMD:R_0805_2012Metric, symbol 2s_Resistor_0805:47k_0805
Connections:
- net 5V en: now also R13.1
- net GND: now also R13.2

Commit message: updates
Parts:
- D1: symbol Diode:MBR0520 -> 2s_diodes:MBR0520; Digi-Key_PN (none) -> MBR0520TPMSTR-ND; MPN (none) -> MBR0520-TP; Manufacturer (none) -> MCC (Micro Commercial Components)
- H1, H2, H3, H4: footprint MountingHole:MountingHole_3.2mm_M3_ISO7380_Pad -> MountingHole:MountingHole_3.2mm_M3_ISO7380
- J5, J6: footprint 2s_connectors:TerminalBlock_MaiXu_MX126-5.0-02P_1x02_P5.00mm -> TerminalBlock_MetzConnect:TerminalBlock_MetzConnect_Type094_RT03502HBLU_1x02_P5.00mm_Horizontal; symbol 2s_connectors:Screw_Terminal_01x02 -> 2s_connectors:screw_terminal_5.00mm; Digi-Key_PN (none) -> A98076-ND; MPN (none) -> 282836-2; Manufacturer (none) -> TE Connectivity AMP Connectors
- U3: symbol Regulator_Switching:LM2733XMF -> 2s_switching_regulators:LM2733XMF; Digi-Key_PN (none) -> LM2733XMF/NOPBTR-ND; MPN (none) -> LM2733XMF/NOPB; Manufacturer (none) -> Texas Instruments
Other:
- company: (none) -> Emmy & Mirco
- title: (none) -> Canda
Changed lines of the file:
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@@
 (kicad_sch
-	(version 20231120)
+	(version 20250114)
 	(generator "eeschema")
-	(generator_version "8.0")
+	(generator_version "9.0")
 	(paper "A3")
+	(title_block
+		(title "Canda")
+		(date "2025-08-20")
+		(rev "v1.0")
+		(company "Emmy & Mirco")
+	)
+	(text "Solenoid"
+		(exclude_from_sim no)
+		(at 47.244 36.068 0)
+		(effects
+			(font
+				(size 1.27 1.27)
+			)
+		)
+	)
 	(junction
 		(at 350.52 40.64)
@@
 		)
 	)
-	(text "Solenoid"
-		(exclude_from_sim no)
-		(at 47.244 36.068 0)
-		(effects
-			(font
-				(size 1.27 1.27)
-			)
-		)
-	)
 	(label "SWDIO"
 		(at 386.08 30.48 0)
-		(fields_autoplaced yes)
 		(effects
 			(font
@@
 	(label "SCL"
 		(at 128.27 64.77 0)
-		(fields_autoplaced yes)
 		(effects
 			(font
@@
 	(label "DBG_TX"
 		(at 262.89 81.28 0)
-		(fields_autoplaced yes)
 		(effects
 			(font
@@
 	(label "SCL"
 		(at 222.25 101.6 0)
-		(fields_autoplaced yes)
 		(effects
 			(font
@@
 	(label "NRST"
 		(at 386.08 40.64 0)
-		(fields_autoplaced yes)
 		(effects
 			(font
@@
 	(label "SDA"
 		(at 128.27 67.31 0)
-		(fields_autoplaced yes)
 		(effects
 			(font
@@
 	(label "DBG_RX"
 		(at 262.89 83.82 0)
-		(fields_autoplaced yes)
 		(effects
 			(font
@@
 	(label "Solenoid En"
 		(at 312.42 149.86 0)
-		(fields_autoplaced yes)
 		(effects
 			(font
@@
 	(label "Solenoid En"
 		(at 262.89 63.5 0)
-		(fields_autoplaced yes)
 		(effects
 			(font
@@
 	(label "5V en"
 		(at 39.37 190.5 0)
-		(fields_autoplaced yes)
 		(effects
 			(font
@@
 	(label "Servo"
 		(at 222.25 88.9 0)
-		(fields_autoplaced yes)
 		(effects
 			(font
@@
 	(label "SDA"
 		(at 222.25 104.14 0)
-		(fields_autoplaced yes)
 		(effects
 			(font
@@
 	(label "DBG_RX"
 		(at 387.35 38.1 0)
-		(fields_autoplaced yes)
 		(effects
 			(font
@@
 	(label "NRST"
 		(at 222.25 58.42 0)
-		(fields_autoplaced yes)
 		(effects
 			(font
@@
 	(label "DBG_TX"
 		(at 356.87 38.1 0)
-		(fields_autoplaced yes)
 		(effects
 			(font
@@
 	(label "SWDIO"
 		(at 262.89 91.44 0)
-		(fields_autoplaced yes)
 		(effects
 			(font
@@
 	(label "SDA"
 		(at 200.66 116.84 0)
-		(fields_autoplaced yes)
 		(effects
 			(font
@@
 	(label "5V en"
 		(at 222.25 86.36 0)
-		(fields_autoplaced yes)
 		(effects
 			(font
@@
 	(label "Servo"
 		(at 368.3 219.71 0)
-		(fields_autoplaced yes)
 		(effects
 			(font
@@
 	(label "SCL"
 		(at 200.66 114.3 0)
-		(fields_autoplaced yes)
 		(effects
 			(font
@@
 	(label "SWCLK"
 		(at 386.08 33.02 0)
-		(fields_autoplaced yes)
 		(effects
 			(font
@@
 	(label "SWCLK"
 		(at 262.89 93.98 0)
-		(fields_autoplaced yes)
 		(effects
 			(font
@@
 	)
 	(symbol
-		(lib_name "Screw_Terminal_01x02_1")
-		(lib_id "2s_connectors:Screw_Terminal_01x02")
+		(lib_id "2s_connectors:screw_terminal_5.00mm")
 		(at 50.8 250.19 180)
 		(unit 1)
@@
 			)
 		)
-		(property "Footprint" "2s_connectors:TerminalBlock_MaiXu_MX126-5.0-02P_1x02_P5.00mm"
-			(at 50.292 258.064 0)
+		(property "Footprint" "TerminalBlock_MetzConnect:TerminalBlock_MetzConnect_Type094_RT03502HBLU_1x02_P5.00mm_Horizontal"
+			(at 50.8 250.19 0)
 			(effects
 				(font
@@
 		)
 		(property "Description" "Generic screw terminal, single row, 01x02, script generated (kicad-library-utils/schlib/autogen/connector/)"
-			(at 50.8 254.508 0)
+			(at 50.8 250.19 0)
+			(effects
+				(font
+					(size 1.27 1.27)
+				)
+				(hide yes)
+			)
+		)
+		(property "MPN" " 282836-2"
+			(at 50.8 250.19 0)
+			(effects
+				(font
+					(size 1.27 1.27)
+				)
+				(hide yes)
+			)
+		)
+		(property "Manufacturer" "TE Connectivity AMP Connectors"
+			(at 50.8 250.19 0)
+			(effects
+				(font
+					(size 1.27 1.27)
+				)
+				(hide yes)
+			)
+		)
+		(property "Digi-Key_PN" "A98076-ND"
+			(at 50.8 250.19 0)
 			(effects
 				(font
@@
 	)
 	(symbol
-		(lib_id "2s_connectors:Screw_Terminal_01x02")
+		(lib_id "2s_connectors:screw_terminal_5.00mm")
 		(at 48.26 43.18 180)
 		(unit 1)
@@
 			)
 		)
-		(property "Footprint" "2s_connectors:TerminalBlock_MaiXu_MX126-5.0-02P_1x02_P5.00mm"
+		(property "Footprint" "TerminalBlock_MetzConnect:TerminalBlock_MetzConnect_Type094_RT03502HBLU_1x02_P5.00mm_Horizontal"
 			(at 48.26 43.18 0)
 			(effects
@@
 			)
 		)
+		(property "MPN" " 282836-2"
+			(at 48.26 43.18 0)
+			(effects
+				(font
+					(size 1.27 1.27)
+				)
+				(hide yes)
+			)
+		)
+		(property "Manufacturer" "TE Connectivity AMP Connectors"
+			(at 48.26 43.18 0)
+			(effects
+				(font
+					(size 1.27 1.27)
+				)
+				(hide yes)
+			)
+		)
+		(property "Digi-Key_PN" "A98076-ND"
+			(at 48.26 43.18 0)
+			(effects
+				(font
+					(size 1.27 1.27)
+				)
+				(hide yes)
+			)
+		)
 		(pin "1"
 		)
@@
 			)
 		)
-		(property "Footprint" "MountingHole:MountingHole_3.2mm_M3_ISO7380_Pad"
+		(property "Footprint" "MountingHole:MountingHole_3.2mm_M3_ISO7380"
 			(at 20.32 107.95 0)
 			(effects
@@
 			)
 		)
-		(property "Footprint" "MountingHole:MountingHole_3.2mm_M3_ISO7380_Pad"
+		(property "Footprint" "MountingHole:MountingHole_3.2mm_M3_ISO7380"
 			(at 20.32 88.9 0)
 			(effects
@@
 			)
 		)
-		(property "Footprint" "MountingHole:MountingHole_3.2mm_M3_ISO7380_Pad"
+		(property "Footprint" "MountingHole:MountingHole_3.2mm_M3_ISO7380"
 			(at 20.32 95.25 0)
 			(effects
@@
 	)
 	(symbol
-		(lib_id "Diode:MBR0520")
+		(lib_id "2s_diodes:MBR0520")
 		(at 354.33 144.78 180)
 		(unit 1)
@@
 			)
 		)
+		(property "Manufacturer" "MCC (Micro Commercial Components)"
+			(at 354.33 144.78 0)
+			(effects
+				(font
+					(size 1.27 1.27)
+				)
+				(hide yes)
+			)
+		)
+		(property "MPN" "MBR0520-TP"
+			(at 354.33 144.78 0)
+			(effects
+				(font
+					(size 1.27 1.27)
+				)
+				(hide yes)
+			)
+		)
+		(property "Digi-Key_PN" "MBR0520TPMSTR-ND"
+			(at 354.33 144.78 0)
+			(effects
+				(font
+					(size 1.27 1.27)
+				)
+				(hide yes)
+			)
+		)
 		(pin "1"
 		)
@@
 	)
 	(symbol
-		(lib_id "Regulator_Switching:LM2733XMF")
+		(lib_id "2s_switching_regulators:LM2733XMF")
 		(at 332.74 147.32 0)
 		(unit 1)
@@
 			)
 		)
+		(property "MPN" "LM2733XMF/NOPB"
+			(at 332.74 147.32 0)
+			(effects
+				(font
+					(size 1.27 1.27)
+				)
+				(hide yes)
+			)
+		)
+		(property "Manufacturer" "Texas Instruments"
+			(at 332.74 147.32 0)
+			(effects
+				(font
+					(size 1.27 1.27)
+				)
+				(hide yes)
+			)
+		)
+		(property "Digi-Key_PN" "LM2733XMF/NOPBTR-ND"
+			(at 332.74 147.32 0)
+			(effects
+				(font
+					(size 1.27 1.27)
+				)
+				(hide yes)
+			)
+		)
 		(pin "3"
 		)
@@
 			)
 		)
-		(property "Footprint" "MountingHole:MountingHole_3.2mm_M3_ISO7380_Pad"
+		(property "Footprint" "MountingHole:MountingHole_3.2mm_M3_ISO7380"
 			(at 20.32 101.6 0)
 			(effects
@@
 		)
 	)
+	(embedded_fonts no)
 )

Commit message: update terminal block
Parts:
- J5, J6: footprint TerminalBlock_MetzConnect:TerminalBlock_MetzConnect_Type094_RT03502HBLU_1x02_P5.00mm_Horizontal -> 2s_connectors:TerminalBlock_MaiXu_MX126-5.0-02P_1x02_P5.00mm; symbol 2s_connectors:screw_terminal_5.00mm -> 2s_connectors:Screw Terminal 5.00mm
Changed lines of the file:
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@@
 	)
 	(symbol
-		(lib_id "2s_connectors:screw_terminal_5.00mm")
+		(lib_id "2s_connectors:Screw Terminal 5.00mm")
 		(at 50.8 250.19 180)
 		(unit 1)
@@
 			)
 		)
-		(property "Footprint" "TerminalBlock_MetzConnect:TerminalBlock_MetzConnect_Type094_RT03502HBLU_1x02_P5.00mm_Horizontal"
+		(property "Footprint" "2s_connectors:TerminalBlock_MaiXu_MX126-5.0-02P_1x02_P5.00mm"
 			(at 50.8 250.19 0)
 			(effects
@@
 	)
 	(symbol
-		(lib_id "2s_connectors:screw_terminal_5.00mm")
+		(lib_id "2s_connectors:Screw Terminal 5.00mm")
 		(at 48.26 43.18 180)
 		(unit 1)
@@
 			)
 		)
-		(property "Footprint" "TerminalBlock_MetzConnect:TerminalBlock_MetzConnect_Type094_RT03502HBLU_1x02_P5.00mm_Horizontal"
+		(property "Footprint" "2s_connectors:TerminalBlock_MaiXu_MX126-5.0-02P_1x02_P5.00mm"
 			(at 48.26 43.18 0)
 			(effects
