File: canda.kicad_sch (KiCad schematic)
At the start: 47 parts, among them J1 2s_cortex-m-10-pin, J3 2x4 male header 2.54 mm, J4 Conn_header_01x04_THT_2.54mm, J5 Screw_Terminal_01x02, J6 Screw_Terminal_01x02, M1 Motor_Servo, Q1 BSS138, Q3 DMG2305UX-13, U1 TPS613222ADBZ, U2 TLV75533PDBVR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

Commit message: add uc bom info
Parts:
- U4: Digi-Key_PN (none) -> 497-17666-2-ND; MPN (none) -> STM32F103C8T6TR; Manufacturer (none) -> STMicroelectronics
Changed lines of the file:
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@@
+			)
+		)
+		(property "Digi-Key_PN" "497-17666-2-ND"
+			(at 245.11 93.98 0)
+			(effects
+				(font
+					(size 1.27 1.27)
+				)
+				(hide yes)
+			)
+		)
+		(property "MPN" "STM32F103C8T6TR"
+			(at 245.11 93.98 0)
+			(effects
+				(font
+					(size 1.27 1.27)
+				)
+				(hide yes)
+			)
+		)
+		(property "Manufacturer" "STMicroelectronics"
+			(at 245.11 93.98 0)
+			(effects
+				(font
+					(size 1.27 1.27)
+				)
+				(hide yes)
 			)
 		)
